Commit message: 修复urdf的问题;添加一些可视化参数

File: source/robot_lab/data/Robots/go2_x5/go2_x5.urdf (robot description, URDF)
Before this commit: robot go2_x5, 50 links, 49 joints
Links:
- link arm_base_link: geometry collision mesh filename=./meshes/X5/base_link.STL; visual mesh filename=./meshes/X5/base_link.STL

Commit message: 取消x5的关节固定;增加机械臂reward;待测试

File: source/robot_lab/data/Robots/go2_x5/go2_x5.urdf (robot description, URDF)
Before this commit: robot go2_x5, 50 links, 49 joints
Joints:
- joint arm_joint1: limit lower=-10 upper=10 effort=100 velocity=1000 -> lower=-2.618 upper=3.14 effort=15 velocity=3; type fixed -> revolute
- joint arm_joint2: limit lower=0 upper=3.14 effort=100 velocity=1000 -> lower=0 upper=3.14 effort=15 velocity=3; type fixed -> revolute
- joint arm_joint3: limit lower=0 upper=3.14 effort=30 velocity=10 -> lower=0 upper=3.14 effort=15 velocity=3; type fixed -> revolute
- joint arm_joint4: limit lower=-1.57079632679 upper=1.57079632679 effort=30 velocity=10 -> lower=-1.5708 upper=1.5708 effort=3 velocity=3; type fixed -> revolute
- joint arm_joint5: limit lower=-1.67 upper=1.67 effort=100 velocity=1000 -> lower=-1.5708 upper=1.5708 effort=3 velocity=3; type fixed -> revolute
- joint arm_joint6: limit lower=-1.57 upper=1.57 effort=100 velocity=1000 -> lower=-1.5708 upper=1.5708 effort=3 velocity=3; type fixed -> revolute
